File: Toxic_Detection_v4.0/power_and_connectors.kicad_sch (KiCad schematic)
At the start: 60 parts, among them IC7 ESDA6V1U1RL, IC8 AP7365-33WG-7, IC9 TPS2054BDR, J10 Conn_01x04_Pin, J11 USB_C_Receptacle, J12 DM3AT-SF-PEJM5, J13 Conn_01x03_Pin, J14 Conn_01x01_Pin, J15 Conn_01x01_Pin, J16 Conn_01x01_Pin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

Commit message: feat: take into account all reviews: add anti-aliasing filters, upgrade 3V3 LDO to support up to 5A, fix UART bug between STM and GNSS
Parts:
- removed C48: 1uF, Capacitor_SMD:C_0805_2012Metric_Pad1.18x1.45mm_HandSolder, symbol Device:C_Small
- removed IC8: AP7365-33WG-7, LDO 3.3V:SOT95P285X130-5N, symbol AP7365-33WG-7:AP7365-33WG-7
- removed J17: Conn_01x01_Pin, Connector_PinSocket_2.54mm:PinSocket_1x01_P2.54mm_Vertical, symbol Connector:Conn_01x01_Pin
- added IC8: AZ1084CD-3.3TRG1, LDO 3.3V:AZ1084CD33TRG1, symbol AZ1084CD-3_3TRG1:AZ1084CD-3.3TRG1
- C46: value 10uF -> 22uF
Connections:
- net +3V3: now also IC8.2 (OUTPUT)
- net GND: now also IC8.1 (GND)
- net VCC: now also IC8.3 (INPUT)
- no-connect marks 18 -> 17
Other:
- moved on the sheet: C46

Commit message: feat: generate gerber, bom, and prepare mouser order
Parts:
- D6: value RED_LED_5mA -> RED_LED_2mA
- R29: value 1k -> 2k
Other:
- note removed: "1k should lead to a 3mA current"
Changed lines of the file:
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@@
 		)
 	)
-	(text "1k should lead to a 3mA current"
+	(text "2k should lead to a 1.5mA current"
 		(exclude_from_sim no)
-		(at 215.9 40.894 0)
+		(at 216.916 40.894 0)
 		(effects
 			(font
@@
 			)
 		)
-		(property "Value" "1k"
+		(property "Value" "2k"
 			(at 207.264 38.1 0)
 			(effects
@@
 			)
 		)
-		(property "Value" "RED_LED_5mA"
+		(property "Value" "RED_LED_2mA"
 			(at 209.55 30.7974 90)
 			(effects
